Commit message: 目前在gazebo中初始状态还算正常，但是站立不起来

File: legged_examples/legged_unitree/quake_description/urdf/quake_without_arm.urdf (robot description, URDF)
Before this commit: robot quake_description, 18 links, 17 joints
Links:
- link LF_FOOT: geometry collision sphere radius=0.022; visual sphere radius=0.032
- link LH_FOOT: geometry collision sphere radius=0.022; visual sphere radius=0.032
- link RF_FOOT: geometry collision sphere radius=0.022; visual sphere radius=0.032
- link RH_FOOT: geometry collision sphere radius=0.022; visual sphere radius=0.032
- link base: geometry collision box size=0.9 0.19 0.05; visual mesh filename=package://quake_description/meshes/trunk.STL scale=1 1 1
